File: Voltage/Voltage.kicad_pcb (KiCad board)
At the start: 2 copper layers, 59.1 x 26.8 mm, 8 parts, among them J1 USB_B_Micro, J2 Screw_Terminal_01x02, U1 AMS1117CD-3.3

Commit message: Complete Voltage converter added bill of materials
Other:
- board text added: "5V to 3.3V"
Changed lines of the file:
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@@
 		(filling no)
 		(pcbplotparams
-			(layerselection 0x00000000_00000000_55555555_5755f5ff)
+			(layerselection 0x00000000_00000000_555555d5_5755ffff)
 			(plot_on_all_layers_selection 0x00000000_00000000_00000000_00000000)
 			(disableapertmacros no)
@@
 			(outputformat 1)
 			(mirror no)
-			(drillshape 1)
+			(drillshape 0)
 			(scaleselection 1)
-			(outputdirectory "")
+			(outputdirectory "gerber/")
 		)
 	)
@@
 			)
 			(justify left bottom)
+		)
+	)
+	(gr_text "5V to 3.3V"
+		(at 93.98 77.47 0)
+		(layer "User.1")
+		(effects
+			(font
+				(size 1 1)
+				(thickness 0.15)
+			)
+			(justify left bottom)
