File: Water alarm Project/Water alarm Project.kicad_pcb (KiCad board)
At the start: 2 copper layers, 39.1 x 38.8 mm, 10 parts, among them J1 Jack-DC, J2 Screw_Terminal_01x02, Q1 2N7000

Commit message: complete water alarm doing final jobs
Parts:
- added G***: LOGO, LOGO, F.Cu at (172.3, 120.7)
- added G***: LOGO, LOGO, F.Cu at (158.7, 122.8)
- added G***: LOGO, LOGO, B.Cu at (158.4, 122.9)
Other:
- board text added: "Water Alarm"
- board text added: "vMay2026"
